Commit message: Update ditto.xacro
updated xacro file

Signed-off-by: SIDDARTH.D <siddarth.dayasagar@gmail.com>

File: ditto_description/urdf/ditto.xacro (robot description, xacro)
@@ -348,10 +348,10 @@
   <child link="fixed_box_1"/>
 </joint>
-<joint name="closing lid" type="prismatic">
+<joint name="closing_lid" type="prismatic">
   <origin xyz="-0.005 0.0 -0.015" rpy="0 0 0"/>
   <parent link="fixed_box_1"/>
   <child link="openingbox_1"/>
   <axis xyz="-1.0 0.0 -0.0"/>
-  <limit upper="0.16" lower="-0.0" effort="100" velocity="100"/>
+  <limit upper="0.16" lower="-0.0" effort="100" velocity="50"/>
 </joint>
 </robot>
