Commit message: Updated laser scan type format - also added octomap but need to test

File: ditto/urdf/ditto.urdf (robot description, URDF)
Before this commit: robot ditto, 3 links, 2 joints
Links:
- added link oak-d-frame
Joints:
- added joint oak-d: type fixed, parent base_footprint, child oak-d-frame, origin xyz=0.12 0.0 0.35 rpy= -1.5707963 0 -1.5707963
